Commit message: refactor

File: urdf/right_open_manipulator.urdf.xacro (robot description, xacro)
@@ -13,5 +13,5 @@
   <!-- World fixed joint-->
   <joint name="world_fixed" type="fixed">
-    <origin xyz="0.1 0 0.5" rpy="0 1.57079632679 0"/>
+    <origin xyz="0.1 0 0.5" rpy="0 -1.57079632679 0"/>
     <parent link="world"/>
     <child link="link1"/>
